File: MPPTLipo.kicad_pcb (KiCad board)
At the start: 2 copper layers, 13 parts, among them IC1 SPV1040, P1 CONN_01X01, P2 SmdPad

Commit message: neu
Parts:
- moved L1 39.1 mm to (141.0, 104.1), turned to 270 degrees
- moved C1 35.2 mm to (153.4, 100.6)
- moved R4 24.5 mm to (155.4, 113.3), turned to 270 degrees
- moved R3 23.8 mm to (156.0, 109.2), turned to 180 degrees
- moved P1 21.7 mm to (151.1, 94.0)
- moved C2 19.7 mm to (157.5, 104.1), turned to 270 degrees
- moved P2 19.4 mm to (157.5, 95.2)
- moved D1 19.1 mm to (149.9, 109.2)
- moved C3 11.4 mm to (167.1, 100.1), turned to 270 degrees
- moved R5 10.3 mm to (157.5, 113.3), turned to 90 degrees
- moved R2 7.73 mm to (161.3, 105.4), turned to 180 degrees
- moved R1 4.58 mm to (161.3, 102.9), turned to 180 degrees
Routing:
- net Net-(C1-Pad1): track 0.00 -> 16.1 mm
- net Net-(D1-Pad1): track 0.00 -> 15.3 mm
- net Net-(C3-Pad2): track 0.00 -> 8.66 mm
- net Net-(C2-Pad1): track 0.00 -> 5.60 mm
- net Net-(C2-Pad2): track 0.00 -> 5.60 mm
Other:
- board outline added: 41.9 x 31.8 mm

Commit message: Lipoprotektionsmodul
Parts:
- added Mod1: Lipo, franzlibtest:LipoProtectPCB, F.Cu at (168.1, 110.2)
- added Mod2: Lipo, franzlibtest:LipoProtectPCB, F.Cu at (177.8, 110.2)
- added P3: P+, Measurement_Points:Measurement_Point_Square-SMD-Pad_Big, F.Cu at (161.5, 91.4)
- added P4: Ü-, Measurement_Points:Measurement_Point_Square-SMD-Pad_Big, F.Cu at (148.8, 90.9)
- P1: value CONN_01X01 -> Solar+; footprint Connectors:1pin -> Measurement_Points:Measurement_Point_Square-SMD-Pad_Big
- P2: value SmdPad -> Solar-; footprint franzlibtest:SmdPadFranz -> Measurement_Points:Measurement_Point_Square-SMD-Pad_Big
- R4: value R -> 10k
- moved P2 4.26 mm to (161.5, 96.5)
- moved P1 2.75 mm to (148.8, 95.5)
Connections:
- D1 pad 1: Net-(D1-Pad1) -> Net-(C3-Pad2)
- D1 pad 2: Net-(C3-Pad2) -> Net-(D1-Pad2)
- IC1 pad 3: Net-(D1-Pad1) -> Net-(D1-Pad2)
- L1 pad 2: Net-(D1-Pad1) -> Net-(D1-Pad2)
Routing:
- net Net-(D1-Pad1): track 15.3 -> 0.00 mm
- net Net-(D1-Pad2): track 0.00 -> 15.2 mm

Commit message: Layout fast fertig
Parts:
- C2, C3: footprint Capacitors_SMD:C_0603_HandSoldering -> Capacitors_SMD:C_0805_HandSoldering
- D1: value D_Schottky -> NSR0530H; footprint Diodes_SMD:D_0805 -> Diodes_SMD:D_SOD-323_HandSoldering
- L1: value L -> 33u; footprint Choke_SMD:Choke_SMD_Wuerth-WE-PD-Typ-LS_Handsoldering -> franzlibtest:VLS6045EX
- R3: value R -> 0.05R; footprint Resistors_SMD:R_0603_HandSoldering -> Resistors_SMD:R_0805_HandSoldering
- moved C3 10.4 mm to (157.0, 98.0)
- moved L1 3.06 mm to (141.2, 101.1)
Routing:
- net Net-(C1-Pad1): track 16.1 -> 2.62 mm
- net Net-(D1-Pad2): track 15.2 -> 8.17 mm
- net Net-(C3-Pad2): track 8.79 -> 7.62 mm
Other:
- net class Default: clearance 0.2 -> 0.1524; trace_width 0.25 -> 0.1524; via_dia 0.6 -> 0.6096; via_drill 0.4 -> 0.1524
- rule trace_clearance: 0.2 -> 0.1524
- rule trace_min: 0.2 -> 0.1524
- rule via_min_drill: 0.3 -> 0.1524
- rule via_min_size: 0.4 -> 0.6096
